File: APDS-9200.brd (EAGLE design)
At the start: 15.2 x 7.6 mm, 9 parts

Commit message: more updates
Parts:
- JMP1, JMP2: device CalvEngIO-Connectors:1X03 -> CalvEngIO-Connectors:1X03@1
Changed lines of the file:
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@@
 <attribute name="NAME" x="9.27075" y="7.006" size="0.508" layer="25" rot="R180" align="top-center"/>
 </element>
-<element name="JMP1" library="CalvEngIO-Connectors" package="1X03" value="JMP-03" x="13.97" y="1.27" smashed="yes" rot="R90"/>
-<element name="JMP2" library="CalvEngIO-Connectors" package="1X03" value="JMP-03" x="1.27" y="1.27" smashed="yes" rot="R90"/>
+<element name="JMP1" library="CalvEngIO-Connectors" package="1X03@1" value="JMP-03" x="13.97" y="1.27" smashed="yes" rot="R90"/>
+<element name="JMP2" library="CalvEngIO-Connectors" package="1X03@1" value="JMP-03" x="1.27" y="1.27" smashed="yes" rot="R90"/>
 <element name="R1" library="CalvEngIO-Passives" package="R0402" value="10k" x="7.62" y="5.74675" smashed="yes" rot="R270"/>
 <element name="R2" library="CalvEngIO-Passives" package="R0402" value="10k" x="9.55675" y="2.286" smashed="yes" rot="R270"/>
